Commit message: Fix audit items, Gazebo traction, and multi-robot readiness
Gazebo physics (verified headless: body now drives straight and turns,
odom vs ground truth within ~4%):
- Ground planes in all worlds had mu=0 (no traction); set to 1.0
- Wheel/caster friction used <surface> blocks that the URDF->SDF parser
  drops; use <mu1>/<mu2> (casters 0.001, wheels 1.0)
- 2 mm caster clearance so the drive wheels carry the load
- VelocityControl plugin (double actuation with ros2_control) is now
  opt-in via use_velocity_control_plugin; its bridge entry disabled

Multi-robot / launch:
- robot_state_publisher.launch: render ros2_controllers.yaml from the
  installed template into a per-robot /tmp file (no hardcoded paths, no
  writes into src); fix enable_odom_tf substitution (never matched)
- xacro takes controllers_file; caster joints honour prefix
- Controller frames prefixed; velocity/accel limits enabled; realistic
  odom covariance
- Controllers started with controller_manager spawners instead of a
  fixed 25 s delay (active in ~4 s)
- Scripts: map path via ros2 pkg prefix; cleanup signals only the
  launch process group instead of pkill -9 on "ros2|gz|..."

Nav2 / code:
- RPP docking_server unified with default params (open_amr_dock)
- Removed dead local static_layer, A* enabled, MPPI allows slow reverse
- cmd_vel_relay: parameterised topics (relative), frame base_footprint
- nav_to_pose: single node, locks/events instead of globals, no
  time.sleep, namespace-aware BasicNavigator
- PoseStampedGenerator is a plain helper taking a clock
- IMU 50 Hz with Gaussian noise; teleop declares use_sim_time
- Package descriptions; open_amr_msgs rosidl_default_generators dep;
  removed placeholder; GitHub Actions CI (build + URDF checks)

Co-Authored-By: Claude Opus 5.5 <noreply@anthropic.com>

File: open_amr_description/urdf/control/gazebo_sim_ros2_control.urdf.xacro (robot description, xacro)
@@ -1,9 +1,9 @@
 <?xml version="1.0" ?>
 <robot xmlns:xacro="http://wiki.ros.org/xacro">
-    <xacro:macro name="load_gazebo_sim_ros2_control_plugin" params="robot_name use_gazebo">
+    <xacro:macro name="load_gazebo_sim_ros2_control_plugin" params="robot_name controllers_file use_gazebo">
         <xacro:if value="${use_gazebo}">
             <gazebo>
                 <plugin filename="gz_ros2_control-system" name="gz_ros2_control::GazeboSimROS2ControlPlugin">
-                    <parameters>$(find open_amr_description)/config/${robot_name}/ros2_controllers.yaml</parameters>
+                    <parameters>${controllers_file}</parameters>
                 </plugin>
             </gazebo>

File: open_amr_description/urdf/mech/caster_wheel.urdf.xacro (robot description, xacro)
@@ -28,17 +28,14 @@
     </link>
     <joint name="${prefix}${name}_caster_joint" type="fixed">
-      <parent link="${parent}"/>
+      <parent link="${prefix}${parent}"/>
       <child link="${prefix}${name}_caster"/>
       <origin xyz="${xyz}" rpy="${rpy}"/>
     </joint>
     <gazebo reference="${prefix}${name}_caster">
-      <surface>
-        <friction>
-          <ode>
-            <mu>0.001</mu>
-            <mu2>0.001</mu2>
-          </ode>
-        </friction>
-      </surface>
+      <!-- URDF->SDF friction must be given as <mu1>/<mu2> directly under <gazebo reference>;
+           a <surface> block here is silently dropped (the caster then brakes with default mu=1).
+           Casters are fixed spheres, so they must be near-frictionless. -->
+      <mu1>0.001</mu1>
+      <mu2>0.001</mu2>
       <visual>
         <material>

File: open_amr_description/urdf/mech/diff_wheel.urdf.xacro (robot description, xacro)
@@ -38,12 +38,7 @@
     </joint>
     <gazebo reference="${prefix}${side}_wheel_link">
-      <surface>
-        <friction>
-          <ode>
-              <mu>1.0</mu>
-              <mu2>0.0</mu2>
-          </ode>
-        </friction>
-      </surface>
+      <!-- <mu1>/<mu2> directly under <gazebo reference> (a <surface> block is dropped by the URDF->SDF parser) -->
+      <mu1>1.0</mu1>
+      <mu2>1.0</mu2>
       <visual>
           <material>

File: open_amr_description/urdf/robots/open_amr.urdf.xacro (robot description, xacro)
@@ -5,9 +5,16 @@
     <xacro:property name="caster_x" value="0.275" />
     <xacro:property name="caster_y" value="0.215" />
-    <xacro:property name="caster_z" value="-0.05" />
+    <!-- 2 mm caster clearance: with all 6 contacts exactly on the ground the base rests on the rigid
+         casters and the drive wheels get ~zero normal force (no traction). Lifting the casters
+         puts the weight on the wheels; the robot rocks <0.5 deg onto one caster pair. -->
+    <xacro:property name="caster_z" value="-0.048" />
     <xacro:property name="caster_radius" value="0.05" />
     <xacro:arg name="robot_name" default="open_amr"/>
     <xacro:arg name="prefix" default=""/>
     <xacro:arg name="use_gazebo" default="false"/>
+    <!-- Rendered by robot_state_publisher.launch.py per robot instance; default = checked-in un-prefixed config -->
+    <xacro:arg name="controllers_file" default="$(find open_amr_description)/config/open_amr/ros2_controllers.yaml"/>
+    <!-- Kinematic body-twist plugin. OFF by default: it double-actuates the robot together with ros2_control -->
+    <xacro:arg name="use_velocity_control_plugin" default="false"/>
     <xacro:include filename="$(find open_amr_description)/urdf/mech/open_amr_base.urdf.xacro"/>
     <xacro:include filename="$(find open_amr_description)/urdf/mech/diff_wheel.urdf.xacro"/>
@@ -54,11 +61,14 @@
       xyz_offset="0 0 0.006"
       rpy_offset="0 0 0"
-      update_rate="15.0"
+      update_rate="50.0"
       topic_name="imu/data"/>
     <xacro:include filename="$(find open_amr_description)/urdf/control/velocity_control_plugin.urdf.xacro" />
-    <xacro:load_velocity_control_plugin use_gazebo="$(arg use_gazebo)"/>
+    <xacro:if value="$(arg use_velocity_control_plugin)">
+      <xacro:load_velocity_control_plugin use_gazebo="$(arg use_gazebo)"/>
+    </xacro:if>
     <xacro:include filename="$(find open_amr_description)/urdf/control/gazebo_sim_ros2_control.urdf.xacro" />
     <xacro:load_gazebo_sim_ros2_control_plugin
       robot_name="$(arg robot_name)"
+      controllers_file="$(arg controllers_file)"
       use_gazebo="$(arg use_gazebo)"/>
     <xacro:include filename="$(find open_amr_description)/urdf/control/open_amr_ros2_control.urdf.xacro" />

File: open_amr_description/urdf/sensors/imu.urdf.xacro (robot description, xacro)
@@ -65,4 +65,9 @@
                 <visualize>${visualize}</visualize>
                 <gz_frame_id>${prefix}${frame_id}_link</gz_frame_id>
+                <!-- Gaussian noise (typical MEMS IMU) so the EKF isn't fed a perfect sensor -->
+                <imu>
+                    <angular_velocity><x><noise type="gaussian"><mean>0.0</mean><stddev>0.0002</stddev></noise></x><y><noise type="gaussian"><mean>0.0</mean><stddev>0.0002</stddev></noise></y><z><noise type="gaussian"><mean>0.0</mean><stddev>0.0002</stddev></noise></z></angular_velocity>
+                    <linear_acceleration><x><noise type="gaussian"><mean>0.0</mean><stddev>0.017</stddev></noise></x><y><noise type="gaussian"><mean>0.0</mean><stddev>0.017</stddev></noise></y><z><noise type="gaussian"><mean>0.0</mean><stddev>0.017</stddev></noise></z></linear_acceleration>
+                </imu>
             </sensor>
         </gazebo>
