Commit message: Phase 4c: robot's own drive and localization stack in Isaac
- open_amr_isaac_hardware: velocity-only joints (AMR wheels): no position
  command interface needed at activation or in the command message
- open_amr_description: URDF arg isaac_ns -> IsaacJointSystem on
  /<ns>/isaac_joint_commands|states
- ekf.yaml: fuse the gyro's yaw rate only (ax at rest reads gravity through
  chassis pitch / mount tilt and walked the filter 0.11 m/min); 50 Hz
- swarm.launch.py: odom_topic for the battery model
- payload_study: chain-rule carton accelerations (a = J qdd + Jdot qd)

Co-Authored-By: Claude Opus 5.5 <noreply@anthropic.com>
Claude-Session: https://claude.ai/code/session_01JGmLjNTMVHeFdAAshqMFWs

File: open_amr_description/urdf/control/open_amr_ros2_control.urdf.xacro (robot description, xacro)
@@ -1,9 +1,16 @@
 <?xml version="1.0" ?>
 <robot xmlns:xacro="http://wiki.ros.org/xacro">
-    <xacro:macro name="open_amr_ros2_control" params="prefix use_gazebo">
+    <!-- hardware: Gazebo (use_gazebo), Isaac Sim (isaac_ns = the robot's namespace: open_amr_isaac_hardware bridged to
+         the simulated wheels, sim/scripts/base_bridge.py), or none here (a real robot's driver brings its own) -->
+    <xacro:macro name="open_amr_ros2_control" params="prefix use_gazebo isaac_ns:=''">
         <ros2_control name="RobotSystem" type="system">
             <hardware>
                 <xacro:if value="${use_gazebo}">
                     <plugin>gz_ros2_control/GazeboSimSystem</plugin>
+                </xacro:if>
+                <xacro:if value="${isaac_ns != ''}">
+                    <plugin>open_amr_isaac_hardware/IsaacJointSystem</plugin>
+                    <param name="joint_commands_topic">/${isaac_ns}/isaac_joint_commands</param>
+                    <param name="joint_states_topic">/${isaac_ns}/isaac_joint_states</param>
                 </xacro:if>
             </hardware>

File: open_amr_description/urdf/robots/open_amr.urdf.xacro (robot description, xacro)
@@ -13,4 +13,5 @@
     <xacro:arg name="prefix" default=""/>
     <xacro:arg name="use_gazebo" default="false"/>
+    <xacro:arg name="isaac_ns" default=""/>   <!-- Isaac Sim with ros2_control (sim real-inputs mode): the namespace of the robot -->
     <!-- Rendered by robot_state_publisher.launch.py per robot instance; default = checked-in un-prefixed config -->
     <xacro:arg name="controllers_file" default="$(find open_amr_description)/config/open_amr/ros2_controllers.yaml"/>
@@ -75,4 +76,5 @@
     <xacro:open_amr_ros2_control
       prefix="$(arg prefix)"
-      use_gazebo="$(arg use_gazebo)"/>
+      use_gazebo="$(arg use_gazebo)"
+      isaac_ns="$(arg isaac_ns)"/>
 </robot>
