Commit message: nanoScan3 pair in the URDF; docking retries re-stage, give up after 3, ACK_FAULT
Co-Authored-By: Claude Opus 5.5 <noreply@anthropic.com>
Claude-Session: https://claude.ai/code/session_01JGmLjNTMVHeFdAAshqMFWs

File: open_amr_description/urdf/robots/open_amr.urdf.xacro (robot description, xacro)
@@ -13,5 +13,8 @@
     <xacro:arg name="prefix" default=""/>
     <xacro:arg name="use_gazebo" default="false"/>
-    <xacro:arg name="isaac_ns" default=""/>   <!-- Isaac Sim with ros2_control (sim real-inputs mode): the namespace of the robot -->
+    <xacro:arg name="isaac_ns" default=""/>
+    <!-- lidar: nanoscan3 = two SICK nanoScan3 safety scanners at diagonal corners (MiR250 layout; the robot's design since
+         2026-10-03: safety-rated, 360 deg); rplidar = the original single RPLIDAR A1M8 (Gazebo stack) -->
+    <xacro:arg name="lidar" default="nanoscan3"/>   <!-- Isaac Sim with ros2_control (sim real-inputs mode): the namespace of the robot -->
     <!-- Rendered by robot_state_publisher.launch.py per robot instance; default = checked-in un-prefixed config -->
     <xacro:arg name="controllers_file" default="$(find open_amr_description)/config/open_amr/ros2_controllers.yaml"/>
@@ -22,4 +25,5 @@
     <xacro:include filename="$(find open_amr_description)/urdf/sensors/rgbd_camera.urdf.xacro"/>
     <xacro:include filename="$(find open_amr_description)/urdf/sensors/lidar.urdf.xacro"/>
+    <xacro:include filename="$(find open_amr_description)/urdf/sensors/nanoscan3.urdf.xacro"/>
     <xacro:include filename="$(find open_amr_description)/urdf/sensors/imu.urdf.xacro"/>
     <xacro:include filename="$(find open_amr_description)/urdf/mech/caster_wheel.urdf.xacro"/>
@@ -47,13 +51,30 @@
       xyz_offset="0.39 0.02 0.042"
       rpy_offset="0 0 0"/>
+    <xacro:if value="${'$(arg lidar)' == 'rplidar'}">
     <xacro:lidar_sensor
-      prefix="$(arg prefix)"
-      parent="base_link"
-      frame_id="laser_frame"
-      xyz_offset="0.320 0 0.12"
-      rpy_offset="0 0 0"
-      mesh_xyz_offset="-0.3 0 -0.22"
-      mesh_rpy_offset="${M_PI/2} 0 0"
-      topic_name="scan"/>
+        prefix="$(arg prefix)"
+        parent="base_link"
+        frame_id="laser_frame"
+        xyz_offset="0.320 0 0.12"
+        rpy_offset="0 0 0"
+        mesh_xyz_offset="-0.3 0 -0.22"
+        mesh_rpy_offset="${M_PI/2} 0 0"
+        topic_name="scan"/>
+    </xacro:if>
+    <xacro:if value="${'$(arg lidar)' == 'nanoscan3'}">
+      <!-- optical centres on the collision outline's corners (x -0.39..0.416, y +-0.319), scan plane 0.12 m above
+           base_link (0.22 m above the floor, as the old lidar), aimed diagonally outward -->
+      <xacro:nanoscan3 prefix="$(arg prefix)" name="front_laser_link" xyz="0.416 0.319 0.12" rpy="0 0 ${M_PI/4}"
+                       topic="scan_front"/>
+      <xacro:nanoscan3 prefix="$(arg prefix)" name="rear_laser_link" xyz="-0.39 -0.319 0.12" rpy="0 0 ${-3*M_PI/4}"
+                       topic="scan_rear"/>
+      <!-- the merged 360 deg scan (dual_laser_merger) for AMCL: a virtual scanner at the base centre, scan height -->
+      <link name="$(arg prefix)scan_merged_link"/>
+      <joint name="$(arg prefix)scan_merged_joint" type="fixed">
+        <parent link="$(arg prefix)base_link"/>
+        <child link="$(arg prefix)scan_merged_link"/>
+        <origin xyz="0 0 0.12" rpy="0 0 0"/>
+      </joint>
+    </xacro:if>
     <xacro:imu_sensor
       prefix="$(arg prefix)"

Commit message: Sensor suite: one nanoScan3 at the nose, D435 moved up, rear ultrasonics; marker tracking in the detector
- URDF lidar:=nanoscan3_front (default): SICK nanoScan3 at x 0.466, scan plane 0.15 m, 230 deg;
  D435 at 0.26 m pitched 20 deg; four rear ultrasonic sensors (park-assist class)
- bay_marker_detector: newest scan only, odometry on its own thread, tracks the marker from
  the last detection + odometry (map-based prediction failed near the bay)

Co-Authored-By: Claude Opus 5.5 <noreply@anthropic.com>
Claude-Session: https://claude.ai/code/session_01JGmLjNTMVHeFdAAshqMFWs

File: open_amr_description/urdf/robots/open_amr.urdf.xacro (robot description, xacro)
@@ -14,7 +14,13 @@
     <xacro:arg name="use_gazebo" default="false"/>
     <xacro:arg name="isaac_ns" default=""/>
-    <!-- lidar: nanoscan3 = two SICK nanoScan3 safety scanners at diagonal corners (MiR250 layout; the robot's design since
-         2026-10-03: safety-rated, 360 deg); rplidar = the original single RPLIDAR A1M8 (Gazebo stack) -->
-    <xacro:arg name="lidar" default="nanoscan3"/>   <!-- Isaac Sim with ros2_control (sim real-inputs mode): the namespace of the robot -->
+    <!-- lidar (notes/Sensor Suite.md):
+         nanoscan3_front = the robot's design (2026-10-03): one SICK nanoScan3 safety scanner at the nose, scan plane
+           150 mm above the floor (ISO 3691-4 / IEC 61496-3: <= 200 mm), 230 deg; the RealSense D435 moved up and
+           tilted down for what the plane misses; rear ultrasonic sensors for backing out of bays (OTTO 100 / Omron LD
+           pattern; the robot only moves forward otherwise)
+         nanoscan3 = two nanoScan3 at diagonal corners (MiR250 layout, 360 deg)
+         rplidar = the original single RPLIDAR A1M8 (Gazebo stack) -->
+    <xacro:arg name="lidar" default="nanoscan3_front"/>
+    <xacro:property name="front_scanner" value="${'$(arg lidar)' == 'nanoscan3_front'}"/>   <!-- Isaac Sim with ros2_control (sim real-inputs mode): the namespace of the robot -->
     <!-- Rendered by robot_state_publisher.launch.py per robot instance; default = checked-in un-prefixed config -->
     <xacro:arg name="controllers_file" default="$(find open_amr_description)/config/open_amr/ros2_controllers.yaml"/>
@@ -46,9 +52,11 @@
     <xacro:caster_wheel prefix="$(arg prefix)" parent="base_link" name="rear_right"
         xyz="${-caster_x} ${-caster_y} ${caster_z}" rpy="0 0 0" radius="${caster_radius}"/>
+    <!-- with the front scanner in the nose, the camera sits above it on the front face, 0.26 m above the floor, tilted
+         20 deg down (floor visible from ~0.35 m ahead, MiR mounts its D435s alike) -->
     <xacro:rgbd_camera
       prefix="$(arg prefix)"
       camera_name="cam_1"
-      xyz_offset="0.39 0.02 0.042"
-      rpy_offset="0 0 0"/>
+      xyz_offset="${'0.42 0 0.16' if front_scanner else '0.39 0.02 0.042'}"
+      rpy_offset="${'0 ' + str(20 * M_PI / 180) + ' 0' if front_scanner else '0 0 0'}"/>
     <xacro:if value="${'$(arg lidar)' == 'rplidar'}">
     <xacro:lidar_sensor
@@ -61,4 +69,31 @@
         mesh_rpy_offset="${M_PI/2} 0 0"
         topic_name="scan"/>
+    </xacro:if>
+    <xacro:if value="${front_scanner}">
+      <!-- optical centre 0.05 m ahead of the nose (x 0.416), on the axis, scan plane 0.05 m above base_link = 0.15 m
+           above the floor; 230 deg: beyond +-115 deg the chassis' central box (+-0.086 m) is in view -->
+      <xacro:nanoscan3 prefix="$(arg prefix)" name="front_laser_link" xyz="0.466 0 0.05" rpy="0 0 0" topic="scan"
+                       fov="${230*M_PI/180}"/>
+      <!-- rear ultrasonic sensors (automotive park-assist class: Bosch USS6 measures 0.15-2.5 m), four across the back
+           at 0.15 m above the floor, the outer two turned 25 deg outward like a car's rear corners: backing out of a
+           bay at <= 0.3 m/s (ISO 3691-4 Table A.1); the robot never reverses elsewhere -->
+      <xacro:macro name="ultrasonic" params="name y yaw">
+        <link name="$(arg prefix)${name}">
+          <visual>
+            <origin xyz="0.005 0 0" rpy="0 ${M_PI/2} 0"/>
+            <geometry><cylinder radius="0.0105" length="0.01"/></geometry>
+            <material name="sonar_white"><color rgba="0.95 0.95 0.95 1"/></material>
+          </visual>
+        </link>
+        <joint name="$(arg prefix)${name}_joint" type="fixed">
+          <parent link="$(arg prefix)base_link"/>
+          <child link="$(arg prefix)${name}"/>
+          <origin xyz="-0.40 ${y} 0.05" rpy="0 0 ${yaw}"/>
+        </joint>
+      </xacro:macro>
+      <xacro:ultrasonic name="us_rear_0" y="0.24" yaw="${M_PI - 25*M_PI/180}"/>
+      <xacro:ultrasonic name="us_rear_1" y="0.08" yaw="${M_PI}"/>
+      <xacro:ultrasonic name="us_rear_2" y="-0.08" yaw="${M_PI}"/>
+      <xacro:ultrasonic name="us_rear_3" y="-0.24" yaw="${M_PI + 25*M_PI/180}"/>
     </xacro:if>
     <xacro:if value="${'$(arg lidar)' == 'nanoscan3'}">
